File: PiLevenMini.sch (KiCad schematic (older format))
At the start: 37 parts, among them IC1 ATMEGA328P-A, J1 RASPBERRY_PI_PLUS_CON, Q1 RJU003N03, Q10 RJU003N03, Q11 RJU003N03, Q2 RJU003N03, Q6 RJU003N03, Q7 BSS84, Q8 BSS84, Q9 RJU003N03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

Commit message: V1.0
Parts:
- added JP?: M08, symbol M08
- added JP?: M10, symbol M10
- added JP?: M07, symbol M07
- added JP?: M06, symbol M06
Connections:
- wire segments 202 -> 227
Other:
- note added: ".1" Breakout for Arduino Pins"
- moved on the sheet: JP1, SJ1, SJ6

Commit message: Refresh schematic, generate PDF
Parts:
- removed JP?: M08, symbol M08
- removed JP?: M10, symbol M10
- removed JP?: M07, symbol M07
- removed JP?: M06, symbol M06
Connections:
- wire segments 227 -> 191
Other:
- note added: "MCU Reset"
- note removed: ".1" Breakout for Arduino Pins"
- note removed: "Reset Circuit"
- moved on the sheet: C12, C13, C14, D1, D2, D3, D4, J1, JP1, Q1, Q10, Q11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

Commit message: V1.1: Fix V1.0 pin assignment problem, minor cleanup
Parts:
- removed SW1: PUSHBUTTON, FT:TACTILE_SWITCH_SMD, symbol SWITCH-MOMENTARY
- added SW1: SW_PUSHBUTTON, symbol SW_PUSHBUTTON
- C10, C11, C12, C13, C14, C16, C9: footprint FT:CAP0603 -> FT:0603_CAP
- IC1: footprint FT:TQFP32-08 -> FT:QFP32_5mm_0.5mm
- Q1, Q10, Q11, Q2, Q6, Q9: footprint FT:SOT323_MOSFET -> FT:SOT323_FET
- Q7, Q8: footprint FT:SOT23_MOSFET -> FT:SOT23_FET
- SHIELD1: value ARDUINO_SHIELD -> ARDUINO_FOOTPRINT; symbol ARDUINO_SHIELD -> ARDUINO_FOOTPRINT
- X1: footprint FT:HC49-US -> FT:CRYSTAL_HC49_PTH
Connections:
- wire segments 191 -> 200
- no-connect marks 26 -> 30
Changed lines of the file:
@@
 EESchema Schematic File Version 2
-LIBS:freetronics_kicad_sch_lib
+LIBS:freetronics_schematic
 LIBS:power
 LIBS:device
@@
 Title "PiLeven Mini"
 Date "Fri 21 Nov 2014"
-Rev ""
+Rev "V1.1"
 Comp "tapr.org/ohl"
 Comment1 "Licensed under TAPR Open Hardware License"
@@
 NoConn ~ 1600 2050
 $Comp
-L ARDUINO_SHIELD SHIELD1
+L ARDUINO_FOOTPRINT SHIELD1
 U 1 1 52A00849
 P 2900 8000
 F 0 "SHIELD1" H 2450 9150 60  0000 C CNN
-F 1 "ARDUINO_SHIELD" H 2950 7050 60  0000 C CNN
+F 1 "ARDUINO_FOOTPRINT" H 2950 7050 60  0000 C CNN
 F 2 "FT:ARDUINO_SHIELD" H 2900 8000 60  0001 C CNN
 F 3 "~" H 2900 8000 60  0000 C CNN
@@
 F 0 "IC1" H 11400 4100 40  0000 L BNN
 F 1 "ATMEGA328P-A" H 12550 1450 40  0000 L BNN
-F 2 "FT:TQFP32-08" H 12150 2850 30  0001 C CIN
+F 2 "FT:QFP32_5mm_0.5mm" H 12150 2850 30  0001 C CIN
 F 3 "~" H 12150 2850 60  0000 C CNN
 	1    12150 2850
@@
 F 0 "C11" H 14300 4050 40  0000 L CNN
 F 1 "22pF" H 14306 3865 40  0000 L CNN
-F 2 "FT:CAP0603" H 14338 3800 30  0001 C CNN
+F 2 "FT:0603_CAP" H 14338 3800 30  0001 C CNN
 F 3 "~" H 14300 3950 60  0000 C CNN
 	1    14300 3950
@@
 F 0 "C10" H 14000 4050 40  0000 L CNN
 F 1 "22pF" H 14006 3865 40  0000 L CNN
-F 2 "FT:CAP0603" H 14038 3800 30  0001 C CNN
+F 2 "FT:0603_CAP" H 14038 3800 30  0001 C CNN
 F 3 "~" H 14000 3950 60  0000 C CNN
 	1    14000 3950
@@
 F 0 "X1" H 14150 3550 60  0000 C CNN
 F 1 "16MHz" H 14150 3250 60  0000 C CNN
-F 2 "FT:HC49-US" H 14150 3400 60  0001 C CNN
+F 2 "FT:CRYSTAL_HC49_PTH" H 14150 3400 60  0001 C CNN
 F 3 "~" H 14150 3400 60  0000 C CNN
 	1    14150 3400
@@
 F 0 "C9" H 10650 3750 40  0000 L CNN
 F 1 "100nF" H 10656 3565 40  0000 L CNN
-F 2 "FT:CAP0603" H 10688 3500 30  0001 C CNN
+F 2 "FT:0603_CAP" H 10688 3500 30  0001 C CNN
 F 3 "~" H 10650 3650 60  0000 C CNN
 	1    10650 3650
@@
 F 0 "Q11" H 8600 7950 70  0000 L BNN
 F 1 "RJU003N03" H 8600 7850 70  0000 L BNN
-F 2 "FT:SOT323_MOSFET" H 8450 8000 60  0001 C CNN
+F 2 "FT:SOT323_FET" H 8450 8000 60  0001 C CNN
 F 3 "~" H 8450 8000 60  0000 C CNN
 	1    8450 8000
@@
 F 0 "Q1" H 5860 2120 60  0000 R CNN
 F 1 "RJU003N03" V 6150 2200 60  0000 R CNN
-F 2 "FT:SOT323_MOSFET" H 5850 1950 60  0001 C CNN
+F 2 "FT:SOT323_FET" H 5850 1950 60  0001 C CNN
 F 3 "~" H 5850 1950 60  0000 C CNN
 	1    5850 1950
@@
 F 0 "Q2" H 5860 3120 60  0000 R CNN
 F 1 "RJU003N03" V 6150 3200 60  0000 R CNN
-F 2 "FT:SOT323_MOSFET" H 5850 2950 60  0001 C CNN
+F 2 "FT:SOT323_FET" H 5850 2950 60  0001 C CNN
 F 3 "~" H 5850 2950 60  0000 C CNN
 	1    5850 2950
@@
 Text Notes 5650 7400 0    79   ~ 0
 Compatible with FTDI cables /\nFreetronics USBSerial
-$Comp
-L SWITCH-MOMENTARY SW1
-U 1 1 53212847
-P 9300 2350
-F 0 "SW1" H 9200 2100 70  0000 L BNN
-F 1 "PUSHBUTTON" H 9100 1950 70  0000 L BNN
-F 2 "FT:TACTILE_SWITCH_SMD" H 9300 2350 60  0001 C CNN
-F 3 "~" H 9300 2350 60  0000 C CNN
-	1    9300 2350
-	0    -1   1    0
-$EndComp
 Text Label 6350 6400 0    60   ~ 0
 CTS
@@
 F 0 "Q6" H 5860 4120 60  0000 R CNN
 F 1 "RJU003N03" V 6150 4200 60  0000 R CNN
-F 2 "FT:SOT323_MOSFET" H 5850 3950 60  0001 C CNN
+F 2 "FT:SOT323_FET" H 5850 3950 60  0001 C CNN
 F 3 "~" H 5850 3950 60  0000 C CNN
 	1    5850 3950
@@
 F 0 "C12" H 7400 4150 40  0000 L CNN
 F 1 "100nF" V 7300 3850 40  0000 L CNN
-F 2 "FT:CAP0603" H 7438 3900 30  0001 C CNN
+F 2 "FT:0603_CAP" H 7438 3900 30  0001 C CNN
 F 3 "~" H 7400 4050 60  0000 C CNN
 	1    7400 4050
 	0    -1   -1   0
 $EndComp
-Text Label 1750 3850 2    60   ~ 0
+Text Label 1700 3350 2    60   ~ 0
 PI_RTS
 $Comp
@@
 F 0 "Q7" H 9860 7720 60  0000 R CNN
 F 1 "BSS84" H 10450 7450 60  0000 R CNN
-F 2 "FT:SOT23_MOSFET" H 9950 7550 60  0001 C CNN
+F 2 "FT:SOT23_FET" H 9950 7550 60  0001 C CNN
 F 3 "~" H 9950 7550 60  0000 C CNN
 	1    9950 7550
@@
 F 0 "C13" H 10400 8050 40  0000 L CNN
 F 1 "1uF" H 10406 7865 40  0000 L CNN
-F 2 "FT:CAP0603" H 10438 7800 30  0001 C CNN
+F 2 "FT:0603_CAP" H 10438 7800 30  0001 C CNN
 F 3 "~" H 10400 7950 60  0000 C CNN
 	1    10400 7950
@@
 F 0 "Q8" H 11860 7720 60  0000 R CNN
 F 1 "BSS84" H 12450 7500 60  0000 R CNN
-F 2 "FT:SOT23_MOSFET" H 11950 7550 60  0001 C CNN
+F 2 "FT:SOT23_FET" H 11950 7550 60  0001 C CNN
 F 3 "~" H 11950 7550 60  0000 C CNN
 	1    11950 7550
@@
 F 0 "C14" H 12400 8050 40  0000 L CNN
 F 1 "1uF" H 12406 7865 40  0000 L CNN
-F 2 "FT:CAP0603" H 12438 7800 30  0001 C CNN
+F 2 "FT:0603_CAP" H 12438 7800 30  0001 C CNN
 F 3 "~" H 12400 7950 60  0000 C CNN
 	1    12400 7950
@@
 F 0 "Q10" H 12860 7920 60  0000 R CNN
 F 1 "RJU003N03" H 13350 7500 60  0000 R CNN
-F 2 "FT:SOT323_MOSFET" H 12950 7750 60  0001 C CNN
+F 2 "FT:SOT323_FET" H 12950 7750 60  0001 C CNN
 F 3 "~" H 12950 7750 60  0000 C CNN
 	1    12950 7750
@@
 F 0 "Q9" H 10860 7920 60  0000 R CNN
 F 1 "RJU003N03" H 11650 7650 60  0000 R CNN
-F 2 "FT:SOT323_MOSFET" H 10950 7750 60  0001 C CNN
+F 2 "FT:SOT323_FET" H 10950 7750 60  0001 C CNN
 F 3 "~" H 10950 7750 60  0000 C CNN
 	1    10950 7750
@@
 F 0 "C16" H 10350 3750 40  0000 L CNN
 F 1 "100nF" H 10356 3565 40  0000 L CNN
-F 2 "FT:CAP0603" H 10388 3500 30  0001 C CNN
+F 2 "FT:0603_CAP" H 10388 3500 30  0001 C CNN
 F 3 "~" H 10350 3650 60  0000 C CNN
 	1    10350 3650
@@
 Wire Wire Line
 	11250 1750 11250 2050
-Wire Wire Line
-	10950 2350 11250 2350
 Connection ~ 11250 4050
 Connection ~ 11250 3950
@@
 	9300 1900 9300 2150
 Wire Wire Line
-	9300 2550 9300 3050
-Wire Wire Line
 	5050 2050 5650 2050
 Wire Wire Line
@@
 Wire Wire Line
 	9100 7650 9100 8300
-Wire Wire Line
-	9300 2150 9400 2150
-Wire Wire Line
-	9300 2550 9400 2550
-Connection ~ 9300 2550
-Connection ~ 9300 2150
 Wire Wire Line
 	7600 4050 7800 4050
@@
 NoConn ~ 1600 3650
 NoConn ~ 1600 3750
-NoConn ~ 1600 3350
+NoConn ~ 1600 3850
 NoConn ~ 1600 3950
 NoConn ~ 1600 4050
@@
 Wire Wire Line
 	13700 3050 13850 3050
+Text Label 3850 7600 0    60   ~ 0
+D11_MOSI
+Text Label 3850 7700 0    60   ~ 0
+D10_~SS
+Text Label 3850 7500 0    60   ~ 0
+D12_MISO
+Text Label 3850 7400 0    60   ~ 0
+D13_SCK
+Wire Wire Line
+	3850 7500 4050 7500
+Wire Wire Line
+	3850 7600 4050 7600
+Wire Wire Line
+	3850 7700 4050 7700
+Wire Wire Line
+	3850 7900 4050 7900
+Wire Wire Line
+	3850 7800 4050 7800
+Wire Wire Line
+	3850 7400 4050 7400
+Text Label 3850 7900 0    60   ~ 0
+D8
+Text Label 3850 7800 0    60   ~ 0
+D9
+Wire Wire Line
+	3850 7300 4450 7300
+Wire Wire Line
+	4450 7300 4450 7450
+$Comp
+L GND #PWR030
+U 1 1 5490C59A
+P 4450 7450
+F 0 "#PWR030" H 4450 7450 30  0001 C CNN
+F 1 "GND" H 4450 7380 30  0001 C CNN
+F 2 "" H 4450 7450 60  0000 C CNN
+F 3 "" H 4450 7450 60  0000 C CNN
+	1    4450 7450
+	1    0    0    -1
+$EndComp
+Wire Wire Line
+	3850 7200 4050 7200
+Wire Wire Line
+	3850 7100 4050 7100
+Wire Wire Line
+	3850 7000 4050 7000
+Text Label 3850 7100 0    60   ~ 0
+A4_SDA
+Text Label 3850 7000 0    60   ~ 0
+A5_SCL
+Text Label 3850 7200 0    60   ~ 0
+AVR_AREF
+NoConn ~ 1750 8100
+NoConn ~ 1600 2250
+NoConn ~ 1600 2350
+NoConn ~ 1600 2450
+Wire Wire Line
+	11250 2350 10850 2350
+$Comp
+L SW_PUSHBUTTON SW1
+U 1 1 54916476
+P 9300 2450
+F 0 "SW1" H 9150 2560 50  0000 C CNN
+F 1 "SW_PUSHBUTTON" H 9300 2370 50  0000 C CNN
+F 2 "" H 9300 2450 60  0000 C CNN
+F 3 "" H 9300 2450 60  0000 C CNN
+	1    9300 2450
+	0    1    1    0
+$EndComp
+Wire Wire Line
+	9300 2750 9300 3050
 $EndSCHEMATC
